Commit message: head stands implemented

File: description/urdf/base.xacro (robot description, xacro)
@@ -114,64 +114,18 @@
         <origin xyz="-${base_width/2 - 0.04} 0 -${sphere_radius + 0.002}" rpy="0 0 0" />
     </joint>
-    <!-- 1. BOYUN (SAĞ-SOL - YAW) -->
-    <link name="neck_yaw_link">
-        <visual>
-            <geometry>
-                <cylinder radius="0.02" length="0.05" />
-            </geometry>
-            <material name="grey" />
-        </visual>
-    </link>
-    <joint name="neck_yaw_joint" type="revolute">
+    <joint name="base_link_rplidar_base_link" type="fixed">
         <parent link="base_link" />
-        <child link="neck_yaw_link" />
-        <origin xyz="0 0 ${base_height}" rpy="0 0 0" /> <!-- Gövdenin tam üst ortası -->
-        <axis xyz="0 0 1" /> <!-- Z ekseninde döner (Sağ-Sol) -->
-        <limit lower="-1.57" upper="1.57" effort="10" velocity="1.0" />
+        <child link="rplidar_base_link" />
+        <origin xyz="${base_width/4} 0 ${base_height-0.005}" rpy="0 0 0" />
     </joint>
-    <!-- 2. BOYUN (YUKARI-AŞAĞI - PITCH) -->
-    <link name="neck_pitch_link">
-        <visual>
-            <geometry>
-                <sphere radius="0.03" />
-            </geometry>
-            <material name="red" />
-        </visual>
-    </link>
-    <joint name="neck_pitch_joint" type="revolute">
-        <parent link="neck_yaw_link" />
-        <child link="neck_pitch_link" />
-        <origin xyz="0 0 0.05" rpy="0 0 0" />
-        <axis xyz="0 1 0" /> <!-- Y ekseninde döner (Yukarı-Aşağı) -->
-        <limit lower="-0.78" upper="0.78" effort="10" velocity="1.0" />
+    <joint name="base_link_rplidar" type="fixed">
+        <parent link="base_link" />
+        <child link="rplidar" />
+        <origin xyz="${base_width/4} 0 ${base_height+0.057}" rpy="0 0 0" />
     </joint>
-    <link name="head_link">
-        <visual>
-            <geometry>
-                <box size="0.06 0.12 0.06" />
-            </geometry>
-            <material name="grey" />
-        </visual>
-    </link>
-    <joint name="head_joint" type="fixed">
-        <parent link="neck_pitch_link" />
-        <child link="head_link" />
-        <origin xyz="0.03 0 0" rpy="0 0 0" />
-    </joint>
-    <link name="left_eye_link">
-        <visual>
-            <geometry>
-                <cylinder radius="0.01" length="0.02" />
-            </geometry>
-            <material name="black" />
-            <origin xyz="0 0 0" rpy="0 ${pi/2} 0" />
-        </visual>
-    </link>
-    <joint name="left_eye_joint" type="revolute">
-        <parent link="head_link" />
-        <child link="left_eye_link" />
-        <origin xyz="0.03 0.03 0" rpy="0 0 0" />
-        <axis xyz="0 0 1" />
-        <limit lower="-0.5" upper="0.5" effort="1" velocity="1.0" />
+    <joint name="base_link_head_base" type="fixed">
+        <parent link="base_link" />
+        <child link="head_base" />
+        <origin xyz="${base_width/4} 0 ${base_height+0.07}" rpy="0 0 0" />
     </joint>
 </robot>

File: description/urdf/denis.urdf.xacro (robot description, xacro)
@@ -12,4 +12,6 @@
     <xacro:include filename="materials.xacro" />
     <xacro:include filename="inertia.xacro" />
+    <xacro:include filename="lidar.xacro" />
+    <xacro:include filename="head.xacro" />
     <xacro:include filename="base.xacro" />
 </robot>

File: description/urdf/materials.xacro (robot description, xacro)
@@ -9,5 +9,5 @@
         <color rgba="0.5 0.5 0.5 1"/>
     </material>
-    <material name="black">
+    <material name="white">
         <color rgba="1 1 1 1"/>
     </material>

Commit message: lidar and diff drive controller movement imp

File: description/urdf/base.xacro (robot description, xacro)
@@ -129,3 +129,11 @@
         <origin xyz="${base_width/4} 0 ${base_height+0.07}" rpy="0 0 0" />
     </joint>
+    <gazebo reference="front_sphere_link">
+        <mu1>0.0</mu1>
+        <mu2>0.0</mu2>
+    </gazebo>
+    <gazebo reference="back_sphere_link">
+        <mu1>0.0</mu1>
+        <mu2>0.0</mu2>
+    </gazebo>
 </robot>

File: description/urdf/lidar.xacro (robot description, xacro)
@@ -1,4 +1,4 @@
 <?xml version="1.0" ?>
-<robot xmlns:xacro="http://www.ros.org/xacro/wiki">
+<robot xmlns:xacro="http://www.ros.org/wiki/xacro">
     <link name="rplidar_base_link">
         <visual>
@@ -10,5 +10,5 @@
         </visual>
         <collision>
-            <origin xxyz="0 0 0" rpy="0 0 0" />
+            <origin xyz="0 0 0" rpy="0 0 0" />
             <geometry>
                 <mesh filename="package://description/mashes/lidar_base.stl" scale="0.001 0.001 0.001" />
@@ -33,3 +33,39 @@
         <xacro:box_inertia m="0.01" x="0.06" y="0.06" z="0.02" o_xyz="0 0 0" o_rpy="0 0 0" />
     </link>
+    <gazebo reference="rplidar">
+        <sensor name="rplidar" type="gpu_lidar">
+            <pose>0 0 0 0 0 0</pose>
+            <topic>scan</topic>
+            <gz_frame_id>rplidar</gz_frame_id>
+            <update_rate>10</update_rate>
+            <always_on>1</always_on>
+            <visualize>true</visualize>
+            <lidar>
+                <scan>
+                    <horizontal>
+                        <samples>360</samples>
+                        <resolution>1</resolution>
+                        <min_angle>-3.14159</min_angle>
+                        <max_angle> 3.14159</max_angle>
+                    </horizontal>
+                    <vertical>
+                        <samples>1</samples>
+                        <resolution>1</resolution>
+                        <min_angle>0</min_angle>
+                        <max_angle>0</max_angle>
+                    </vertical>
+                </scan>
+                <range>
+                    <min>0.15</min>
+                    <max>12.0</max>
+                    <resolution>0.01</resolution>
+                </range>
+                <noise>
+                    <type>gaussian</type>
+                    <mean>0.0</mean>
+                    <stddev>0.01</stddev>
+                </noise>
+            </lidar>
+        </sensor>
+    </gazebo>
 </robot>
