Commit message: hotfix and enchan

File: description/urdf/head.xacro (robot description, xacro)
@@ -5,5 +5,5 @@
             <origin xyz="0 0 0" rpy="0 0 0" />
             <geometry>
-                <mesh filename="package://description/mashes/head_base.stl"
+                <mesh filename="package://description/meshes/head_base.stl"
                     scale="0.001 0.001 0.001" />
             </geometry>
@@ -13,5 +13,5 @@
             <origin xyz="0 0 0" rpy="0 0 0" />
             <geometry>
-                <mesh filename="package://description/mashes/head_base.stl"
+                <mesh filename="package://description/meshes/head_base.stl"
                     scale="0.001 0.001 0.001" />
             </geometry>

File: description/urdf/lidar.xacro (robot description, xacro)
@@ -5,5 +5,5 @@
             <origin xyz="0 0 0" rpy="0 0 0" />
             <geometry>
-                <mesh filename="package://description/mashes/lidar_base.stl" scale="0.001 0.001 0.001" />
+                <mesh filename="package://description/meshes/lidar_base.stl" scale="0.001 0.001 0.001" />
             </geometry>
             <material name="white" />
@@ -12,5 +12,5 @@
             <origin xyz="0 0 0" rpy="0 0 0" />
             <geometry>
-                <mesh filename="package://description/mashes/lidar_base.stl" scale="0.001 0.001 0.001" />
+                <mesh filename="package://description/meshes/lidar_base.stl" scale="0.001 0.001 0.001" />
             </geometry>
         </collision>
