Commit message: head movement imp

File: description/ros2_control/ros2_control.xacro (robot description, xacro)
@@ -21,4 +21,20 @@
                 <state_interface name="velocity" />
                 <state_interface name="position" />
+            </joint>
+            <joint name="head_base_neck_pan_link">
+                <command_interface name="position">
+                    <param name="min">-3.14159</param>
+                    <param name="max">3.14159</param>
+                </command_interface>
+                <state_interface name="position" />
+                <state_interface name="velocity" />
+            </joint>
+            <joint name="head_base_tilt_pan_link">
+                <command_interface name="position">
+                    <param name="min">-3.14159</param>
+                    <param name="max">3.14159</param>
+                </command_interface>
+                <state_interface name="position" />
+                <state_interface name="velocity" />
             </joint>
         </ros2_control>

File: description/urdf/head.xacro (robot description, xacro)
@@ -1,3 +1,3 @@
-<?xml version="1.0" ?>
+<?xml version="1.0"?>
 <robot xmlns:xacro="http://www.ros.org/wiki/xacro">
     <link name="head_base">
@@ -5,5 +5,6 @@
             <origin xyz="0 0 0" rpy="0 0 0" />
             <geometry>
-                <mesh filename="package://description/mashes/head_base.stl" scale="0.001 0.001 0.001"/>
+                <mesh filename="package://description/mashes/head_base.stl"
+                    scale="0.001 0.001 0.001" />
             </geometry>
             <material name="white" />
@@ -12,8 +13,104 @@
             <origin xyz="0 0 0" rpy="0 0 0" />
             <geometry>
-                <mesh filename="package://description/mashes/head_base.stl" scale="0.001 0.001 0.001"/>
+                <mesh filename="package://description/mashes/head_base.stl"
+                    scale="0.001 0.001 0.001" />
             </geometry>
         </collision>
         <xacro:box_inertia m="0.11" x="0.16" y="0.16" z="0.03540" o_xyz="0 0 0" o_rpy="0 0 0" />
     </link>
+    <link name="neck_pan_link">
+        <visual>
+            <origin xyz="0 0 0.04" rpy="0 0 0" />
+            <geometry>
+                <box size="0.04 0.04 0.08" />
+            </geometry>
+            <material name="red" />
+        </visual>
+        <collision>
+            <origin xyz="0 0 0.04" rpy="0 0 0" />
+            <geometry>
+                <box size="0.04 0.04 0.08" />
+            </geometry>
+        </collision>
+        <xacro:box_inertia m="0.02" x="0.04" y="0.04" z="0.08" o_xyz="0 0 0.04" o_rpy="0 0 0" />
+    </link>
+    <link name="neck_tilt_link">
+        <visual>
+            <origin xyz="0 0 0" rpy="0 0 0" />
+            <geometry>
+                <box size="0.08 0.08 0.02" />
+            </geometry>
+            <material name="white" />
+        </visual>
+        <collision>
+            <origin xyz="0 0 0" rpy="0 0 0" />
+            <geometry>
+                <box size="0.08 0.08 0.02" />
+            </geometry>
+        </collision>
+        <xacro:box_inertia m="0.01" x="0.08" y="0.08" z="0.02" o_xyz="0 0 0" o_rpy="0 0 0" />
+    </link>
+    <link name="camera_link">
+        <visual>
+            <origin xyz="0 0 0" rpy="0 0 0" />
+            <geometry>
+                <box size="0.03 0.06 0.03" />
+            </geometry>
+            <material name="red" />
+        </visual>
+        <collision>
+            <origin xyz="0 0 0" rpy="0 0 0" />
+            <geometry>
+                <box size="0.03 0.06 0.03" />
+            </geometry>
+        </collision>
+        <xacro:box_inertia m="0.01" x="0.03" y="0.06" z="0.03" o_xyz="0 0 0" o_rpy="0 0 0" />
+    </link>
+    <joint name="head_base_neck_pan_link" type="revolute">
+        <parent link="head_base" />
+        <child link="neck_pan_link" />
+        <origin xyz="0 0 0.02" rpy="0 0 0" />
+        <limit lower="-${pi}" upper="${pi}" effort="100" velocity="100" />
+        <axis xyz="0 0 1" />
+    </joint>
+    <joint name="head_base_tilt_pan_link" type="revolute">
+        <parent link="neck_pan_link" />
+        <child link="neck_tilt_link" />
+        <origin xyz="0 0 0.08" rpy="0 0 0" />
+        <limit lower="-${pi}" upper="${pi}" effort="100" velocity="100" />
+        <axis xyz="0 1 0" />
+        <dynamics damping="2.0" friction="1.0" />
+    </joint>
+    <joint name="neck_tilt_camera_joint" type="fixed">
+        <parent link="neck_tilt_link" />
+        <child link="camera_link" />
+        <origin xyz="0.08 0 0" rpy="0 0 0" />
+    </joint>
+    <gazebo reference="camera_link">
+        <sensor name="camera" type="camera">
+            <pose>0 0 0 0 0 0</pose>
+            <topic>camera/image_raw</topic>
+            <gz_frame_id>camera_link</gz_frame_id>
+            <update_rate>30</update_rate>
+            <always_on>1</always_on>
+            <visualize>true</visualize>
+            <camera>
+                <horizontal_fov>1.047</horizontal_fov>
+                <image>
+                    <width>640</width>
+                    <height>480</height>
+                    <format>R8G8B8</format>
+                </image>
+                <clip>
+                    <near>0.1</near>
+                    <far>100</far>
+                </clip>
+                <noise>
+                    <type>gaussian</type>
+                    <mean>0.0</mean>
+                    <stddev>0.007</stddev>
+                </noise>
+            </camera>
+        </sensor>
+    </gazebo>
 </robot>
